File: LedScoreBoard/LedAnodeDrivers.kicad_sch (KiCad schematic)
At the start: 27 parts

Commit message: 回路図更新
Parts:
- gave numbers to parts that had none: 27

Commit message: パターン完成
Parts:
- D202, D203, D204: footprint Diode_THT:D_DO-27_P5.08mm_Vertical_AnodeUp -> Diode_THT:D_DO-27_P12.70mm_Horizontal
Changed lines of the file:
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@@
     (property "Reference" "D203" (id 0) (at 191.77 92.71 0))
     (property "Value" "ER504" (id 1) (at 191.77 95.25 0))
-    (property "Footprint" "Diode_THT:D_DO-27_P5.08mm_Vertical_AnodeUp" (id 2) (at 191.77 99.06 0)
+    (property "Footprint" "Diode_THT:D_DO-27_P12.70mm_Horizontal" (id 2) (at 191.77 99.06 0)
       (effects (font (size 1.27 1.27)) hide)
     )
@@
     (property "Reference" "D202" (id 0) (at 191.77 48.26 0))
     (property "Value" "ER504" (id 1) (at 191.77 50.8 0))
-    (property "Footprint" "Diode_THT:D_DO-27_P5.08mm_Vertical_AnodeUp" (id 2) (at 191.77 54.61 0)
+    (property "Footprint" "Diode_THT:D_DO-27_P12.70mm_Horizontal" (id 2) (at 191.77 54.61 0)
       (effects (font (size 1.27 1.27)) hide)
     )
@@
     (property "Reference" "D204" (id 0) (at 191.77 137.16 0))
     (property "Value" "ER504" (id 1) (at 191.77 139.7 0))
-    (property "Footprint" "Diode_THT:D_DO-27_P5.08mm_Vertical_AnodeUp" (id 2) (at 191.77 143.51 0)
-      (effects (font (size 1.27 1.27)) hide)
-    )
+    (property "Footprint" "Diode_THT:D_DO-27_P12.70mm_Horizontal" (id 2) (at 191.77 143.51 0)
+      (effects (font (size 1.27 1.27)) hide)
+    )

Commit message: 回路修正
Parts:
- D202, D203, D204: footprint Diode_THT:D_DO-27_P12.70mm_Horizontal -> Diode_THT:D_DO-27_P15.24mm_Horizontal
Changed lines of the file:
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@@
     (property "Reference" "D203" (id 0) (at 191.77 92.71 0))
     (property "Value" "ER504" (id 1) (at 191.77 95.25 0))
-    (property "Footprint" "Diode_THT:D_DO-27_P12.70mm_Horizontal" (id 2) (at 191.77 99.06 0)
+    (property "Footprint" "Diode_THT:D_DO-27_P15.24mm_Horizontal" (id 2) (at 191.77 99.06 0)
       (effects (font (size 1.27 1.27)) hide)
     )
@@
   (symbol (lib_id "power:GND") (at 127 152.4 0) (unit 1)
     (in_bom yes) (on_board yes) (fields_autoplaced)
-    (property "Reference" "#PWR0205" (id 0) (at 127 158.75 0)
+    (property "Reference" "#PWR0202" (id 0) (at 127 158.75 0)
       (effects (font (size 1.27 1.27)) hide)
     )
@@
     (property "Reference" "D202" (id 0) (at 191.77 48.26 0))
     (property "Value" "ER504" (id 1) (at 191.77 50.8 0))
-    (property "Footprint" "Diode_THT:D_DO-27_P12.70mm_Horizontal" (id 2) (at 191.77 54.61 0)
+    (property "Footprint" "Diode_THT:D_DO-27_P15.24mm_Horizontal" (id 2) (at 191.77 54.61 0)
       (effects (font (size 1.27 1.27)) hide)
     )
@@
   (symbol (lib_id "power:GND") (at 143.51 64.77 0) (unit 1)
     (in_bom yes) (on_board yes) (fields_autoplaced)
-    (property "Reference" "#PWR0202" (id 0) (at 143.51 71.12 0)
+    (property "Reference" "#PWR0205" (id 0) (at 143.51 71.12 0)
       (effects (font (size 1.27 1.27)) hide)
     )
@@
     (property "Reference" "D204" (id 0) (at 191.77 137.16 0))
     (property "Value" "ER504" (id 1) (at 191.77 139.7 0))
-    (property "Footprint" "Diode_THT:D_DO-27_P12.70mm_Horizontal" (id 2) (at 191.77 143.51 0)
+    (property "Footprint" "Diode_THT:D_DO-27_P15.24mm_Horizontal" (id 2) (at 191.77 143.51 0)
       (effects (font (size 1.27 1.27)) hide)
     )
@@
   (symbol (lib_id "power:GND") (at 127 63.5 0) (unit 1)
     (in_bom yes) (on_board yes) (fields_autoplaced)
-    (property "Reference" "#PWR0201" (id 0) (at 127 69.85 0)
+    (property "Reference" "#PWR0203" (id 0) (at 127 69.85 0)
       (effects (font (size 1.27 1.27)) hide)
     )
@@
   (symbol (lib_id "power:VDD") (at 186.69 27.94 0) (unit 1)
     (in_bom yes) (on_board yes) (fields_autoplaced)
-    (property "Reference" "#PWR0203" (id 0) (at 186.69 31.75 0)
-      (effects (font (size 1.27 1.27)) hide)
-    )
+    (property "Reference" "#PWR0201" (id 0) (at 186.69 31.75 0)
+      (effects (font (size 1.27 1.27)) hide)
+    )

Commit message: ver2完成
Parts:
- added H201, H202, H203: MountingHole, MountingHole:MountingHole_2.2mm_M2, symbol Mechanical:MountingHole
Changed lines of the file:
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@@
     (pin "3")
+  )
+  (symbol (lib_id "Mechanical:MountingHole") (at 100.33 179.07 0) (unit 1)
+    (in_bom yes) (on_board yes) (fields_autoplaced)
+    (property "Reference" "H201" (id 0) (at 102.87 177.7999 0)
+      (effects (font (size 1.27 1.27)) (justify left))
+    )
+    (property "Value" "MountingHole" (id 1) (at 102.87 180.3399 0)
+      (effects (font (size 1.27 1.27)) (justify left))
+    )
+    (property "Footprint" "MountingHole:MountingHole_2.2mm_M2" (id 2) (at 100.33 179.07 0)
+      (effects (font (size 1.27 1.27)) hide)
+    )
+    (property "Datasheet" "~" (id 3) (at 100.33 179.07 0)
+      (effects (font (size 1.27 1.27)) hide)
+    )
   )
   (symbol (lib_id "power:GND") (at 127 152.4 0) (unit 1)
@@
     (pin "3")
   )
+  (symbol (lib_id "Mechanical:MountingHole") (at 100.33 185.42 0) (unit 1)
+    (in_bom yes) (on_board yes) (fields_autoplaced)
+    (property "Reference" "H202" (id 0) (at 102.87 184.1499 0)
+      (effects (font (size 1.27 1.27)) (justify left))
+    )
+    (property "Value" "MountingHole" (id 1) (at 102.87 186.6899 0)
+      (effects (font (size 1.27 1.27)) (justify left))
+    )
+    (property "Footprint" "MountingHole:MountingHole_2.2mm_M2" (id 2) (at 100.33 185.42 0)
+      (effects (font (size 1.27 1.27)) hide)
+    )
+    (property "Datasheet" "~" (id 3) (at 100.33 185.42 0)
+      (effects (font (size 1.27 1.27)) hide)
+    )
+  )
   (symbol (lib_id "Device:Q_PMOS_GDS") (at 184.15 130.81 0) (mirror x) (unit 1)
     (in_bom yes) (on_board yes) (fields_autoplaced)
@@
     (pin "1")
   )
+  (symbol (lib_id "Mechanical:MountingHole") (at 100.33 191.77 0) (unit 1)
+    (in_bom yes) (on_board yes) (fields_autoplaced)
+    (property "Reference" "H203" (id 0) (at 102.87 190.4999 0)
+      (effects (font (size 1.27 1.27)) (justify left))
+    )
+    (property "Value" "MountingHole" (id 1) (at 102.87 193.0399 0)
+      (effects (font (size 1.27 1.27)) (justify left))
+    )
+    (property "Footprint" "MountingHole:MountingHole_2.2mm_M2" (id 2) (at 100.33 191.77 0)
+      (effects (font (size 1.27 1.27)) hide)
+    )
+    (property "Datasheet" "~" (id 3) (at 100.33 191.77 0)
+      (effects (font (size 1.27 1.27)) hide)
+    )
+  )
   (symbol (lib_id "power:VDD") (at 186.69 116.84 0) (unit 1)
