File: LedScoreBoard/LedCathodeDrivers.kicad_sch (KiCad schematic)
At the start: 57 parts

Commit message: 回路図更新
Parts:
- removed C? (x5): C, symbol Device:C
- added C302, C303, C304, C305, C306, C307: 1u, Capacitor_SMD:C_0603_1608Metric, symbol Device:C
- C301: renamed from C?; value C -> 1u; footprint (none) -> Capacitor_SMD:C_0603_1608Metric
- gave numbers to parts that had none: 48
Connections:
- net CsensB: now also C302.1
- net CsensC: now also C303.1
- net CsensD: now also C304.1
- net CsensE: now also C305.1
- net CsensF: now also C306.1
- net CsensG: now also C307.1
- net GND: now also C302.2, C303.2, C304.2, C305.2, C306.2, C307.2

Commit message: 配置ブロック決定
Parts:
- renumbered U302 to U301, U306 to U301, U301 to U302, U303 to U302, U307 to U302, U304 to U303, U308 to U303, U309 to U304, U305 to U304
Connections:
- net CsensA: now also U301.6 (-); no longer U301.2 (-)
- net CsensB: now also U302.2 (-); no longer U302.6 (-)
- net CsensC: now also U302.6 (-); no longer U302.2 (-)
- net CsensD: now also U303.2 (-); no longer U303.6 (-)
- net CsensE: now also U303.6 (-); no longer U303.2 (-)
- net CsensF: now also U304.2 (-); no longer U304.6 (-)
- net CsensG: now also U304.6 (-); no longer U304.2 (-)
- net at R316.1: now also U304.1; no longer U304.7
- net at R301.1: now also U301.7; no longer U301.1
- net at Q301.2 (S): now also U301.5 (+); no longer U301.3 (+)
- net at R313.1: now also U303.7; no longer U303.1
- net at Q303.2 (S): now also U302.3 (+); no longer U302.5 (+)
- net at R304.1: now also U302.1; no longer U302.7
- net at Q311.2 (S): now also U304.3 (+); no longer U304.5 (+)
- net at Q307.2 (S): now also U303.3 (+); no longer U303.5 (+)
- net at R310.1: now also U303.1; no longer U303.7
- net at Q309.2 (S): now also U303.5 (+); no longer U303.3 (+)
- net at R307.1: now also U302.7; no longer U302.1
- net at Q305.2 (S): now also U302.5 (+); no longer U302.3 (+)
- net at R319.1: now also U304.7; no longer U304.1
- net at Q313.2 (S): now also U304.5 (+); no longer U304.3 (+)
Changed lines of the file:
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@@
   (symbol (lib_id "Amplifier_Operational:LM358") (at 99.06 167.64 0) (unit 3)
     (in_bom yes) (on_board yes) (fields_autoplaced)
-    (property "Reference" "U309" (id 0) (at 97.79 166.3699 0)
+    (property "Reference" "U304" (id 0) (at 97.79 166.3699 0)
       (effects (font (size 1.27 1.27)) (justify left))
     )
@@
     (pin "1")
   )
-  (symbol (lib_id "Amplifier_Operational:LM358") (at 107.95 45.72 0) (unit 1)
-    (in_bom yes) (on_board yes) (fields_autoplaced)
-    (property "Reference" "U302" (id 0) (at 107.95 35.56 0))
+  (symbol (lib_id "Amplifier_Operational:LM358") (at 107.95 45.72 0) (unit 2)
+    (in_bom yes) (on_board yes) (fields_autoplaced)
+    (property "Reference" "U301" (id 0) (at 107.95 35.56 0))
     (property "Value" "LM358" (id 1) (at 107.95 38.1 0))
     (property "Footprint" "Package_SO:TSSOP-8_3x3mm_P0.65mm" (id 2) (at 107.95 45.72 0)
@@
     (pin "3")
   )
-  (symbol (lib_id "Amplifier_Operational:LM358") (at 172.72 45.72 0) (unit 2)
-    (in_bom yes) (on_board yes) (fields_autoplaced)
-    (property "Reference" "U301" (id 0) (at 172.72 35.56 0))
+  (symbol (lib_id "Amplifier_Operational:LM358") (at 172.72 45.72 0) (unit 1)
+    (in_bom yes) (on_board yes) (fields_autoplaced)
+    (property "Reference" "U302" (id 0) (at 172.72 35.56 0))
     (property "Value" "LM358" (id 1) (at 172.72 38.1 0))
     (property "Footprint" "Package_SO:TSSOP-8_3x3mm_P0.65mm" (id 2) (at 172.72 45.72 0)
@@
     (pin "2")
   )
-  (symbol (lib_id "Amplifier_Operational:LM358") (at 172.72 111.76 0) (unit 2)
-    (in_bom yes) (on_board yes) (fields_autoplaced)
-    (property "Reference" "U305" (id 0) (at 172.72 101.6 0))
+  (symbol (lib_id "Amplifier_Operational:LM358") (at 172.72 111.76 0) (unit 1)
+    (in_bom yes) (on_board yes) (fields_autoplaced)
+    (property "Reference" "U304" (id 0) (at 172.72 101.6 0))
     (property "Value" "LM358" (id 1) (at 172.72 104.14 0))
     (property "Footprint" "Package_SO:TSSOP-8_3x3mm_P0.65mm" (id 2) (at 172.72 111.76 0)
@@
     (pin "2")
   )
-  (symbol (lib_id "Amplifier_Operational:LM358") (at 44.45 111.76 0) (unit 2)
-    (in_bom yes) (on_board yes) (fields_autoplaced)
-    (property "Reference" "U304" (id 0) (at 44.45 101.6 0))
+  (symbol (lib_id "Amplifier_Operational:LM358") (at 44.45 111.76 0) (unit 1)
+    (in_bom yes) (on_board yes) (fields_autoplaced)
+    (property "Reference" "U303" (id 0) (at 44.45 101.6 0))
     (property "Value" "LM358" (id 1) (at 44.45 104.14 0))
     (property "Footprint" "Package_SO:TSSOP-8_3x3mm_P0.65mm" (id 2) (at 44.45 111.76 0)
@@
     (pin "8")
   )
-  (symbol (lib_id "Amplifier_Operational:LM358") (at 107.95 111.76 0) (unit 1)
-    (in_bom yes) (on_board yes) (fields_autoplaced)
-    (property "Reference" "U304" (id 0) (at 107.95 101.6 0))
+  (symbol (lib_id "Amplifier_Operational:LM358") (at 107.95 111.76 0) (unit 2)
+    (in_bom yes) (on_board yes) (fields_autoplaced)
+    (property "Reference" "U303" (id 0) (at 107.95 101.6 0))
     (property "Value" "LM358" (id 1) (at 107.95 104.14 0))
     (property "Footprint" "Package_SO:TSSOP-8_3x3mm_P0.65mm" (id 2) (at 107.95 111.76 0)
@@
     (pin "2")
   )
-  (symbol (lib_id "Amplifier_Operational:LM358") (at 240.03 45.72 0) (unit 1)
-    (in_bom yes) (on_board yes) (fields_autoplaced)
-    (property "Reference" "U303" (id 0) (at 240.03 35.56 0))
+  (symbol (lib_id "Amplifier_Operational:LM358") (at 240.03 45.72 0) (unit 2)
+    (in_bom yes) (on_board yes) (fields_autoplaced)
+    (property "Reference" "U302" (id 0) (at 240.03 35.56 0))
     (property "Value" "LM358" (id 1) (at 240.03 38.1 0))
     (property "Footprint" "Package_SO:TSSOP-8_3x3mm_P0.65mm" (id 2) (at 240.03 45.72 0)
@@
   (symbol (lib_id "Amplifier_Operational:LM358") (at 81.28 167.64 0) (unit 3)
     (in_bom yes) (on_board yes) (fields_autoplaced)
-    (property "Reference" "U307" (id 0) (at 80.01 166.3699 0)
+    (property "Reference" "U302" (id 0) (at 80.01 166.3699 0)
       (effects (font (size 1.27 1.27)) (justify left))
     )
@@
     (pin "2")
   )
-  (symbol (lib_id "Amplifier_Operational:LM358") (at 240.03 111.76 0) (unit 1)
-    (in_bom yes) (on_board yes) (fields_autoplaced)
-    (property "Reference" "U305" (id 0) (at 240.03 101.6 0))
+  (symbol (lib_id "Amplifier_Operational:LM358") (at 240.03 111.76 0) (unit 2)
+    (in_bom yes) (on_board yes) (fields_autoplaced)
+    (property "Reference" "U304" (id 0) (at 240.03 101.6 0))
     (property "Value" "LM358" (id 1) (at 240.03 104.14 0))
     (property "Footprint" "Package_SO:TSSOP-8_3x3mm_P0.65mm" (id 2) (at 240.03 111.76 0)
@@
   (symbol (lib_id "Amplifier_Operational:LM358") (at 72.39 167.64 0) (unit 3)
     (in_bom yes) (on_board yes) (fields_autoplaced)
-    (property "Reference" "U306" (id 0) (at 71.12 166.3699 0)
+    (property "Reference" "U301" (id 0) (at 71.12 166.3699 0)
       (effects (font (size 1.27 1.27)) (justify left))
     )
@@
   (symbol (lib_id "Amplifier_Operational:LM358") (at 90.17 167.64 0) (unit 3)
     (in_bom yes) (on_board yes) (fields_autoplaced)
-    (property "Reference" "U308" (id 0) (at 88.9 166.3699 0)
-      (effects (font (size 1.27 1.27)) (justify left))
-    )
+    (property "Reference" "U303" (id 0) (at 88.9 166.3699 0)
+      (effects (font (size 1.27 1.27)) (justify left))
+    )

Commit message: Vref修正
Connections:
- net Vref: no longer U301.3 (+)
- new net VrefIn: U301.3 (+)
Changed lines of the file:
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@@
     (effects (font (size 1.27 1.27)) (justify right))
   )
-  (hierarchical_label "Vref" (shape input) (at 31.75 43.18 180)
+  (hierarchical_label "VrefIn" (shape input) (at 31.75 43.18 180)
     (effects (font (size 1.27 1.27)) (justify right))
   )

Commit message: 回路修正
Parts:
- added R301, R305, R309, R313, R317, R321, R325: 10k, Resistor_SMD:R_0603_1608Metric, symbol Device:R
- U301, U302, U303, U304: footprint Package_SO:TSSOP-8_3x3mm_P0.65mm -> Package_SO:SOP-8_3.9x4.9mm_P1.27mm
- renumbered R301 to R302, R302 to R303, R303 to R304, R304 to R306, R305 to R307, R306 to R308, R307 to R310, R308 to R311, R309 to R312, R310 to R314, R311 to R315, R312 to R316, R313 to R318, R314 to R319, R315 to R320, R316 to R322, R317 to R323, R318 to R324, R319 to R326, R320 to R327, R321 to R328
Connections:
- net GND: now also R301.2, R305.2, R309.2, R313.2, R317.2, R321.2, R325.2
- net at Q301.2 (S), U301.5 (+): now also R301.1
- net at Q303.2 (S), U302.3 (+): now also R305.1
- net at Q311.2 (S), U304.3 (+): now also R321.1
- net at Q307.2 (S), U303.3 (+): now also R313.1
- net at Q309.2 (S), U303.5 (+): now also R317.1
- net at Q305.2 (S), U302.5 (+): now also R309.1
- net at Q313.2 (S), U304.5 (+): now also R325.1

Commit message: ver2完成
Parts:
- added H301, H302, H303, H304, H305, H306, H307: MountingHole, MountingHole:MountingHole_2.2mm_M2, symbol Mechanical:MountingHole
Connections:
- net VrefIn renamed PicVref
Changed lines of the file:
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@@
     (effects (font (size 1.27 1.27)) (justify right))
   )
-  (hierarchical_label "VrefIn" (shape input) (at 31.75 43.18 180)
+  (hierarchical_label "PicVref" (shape input) (at 31.75 43.18 180)
     (effects (font (size 1.27 1.27)) (justify right))
   )
@@
     (pin "1")
     (pin "2")
+  )
+  (symbol (lib_id "Mechanical:MountingHole") (at 257.81 153.67 0) (unit 1)
+    (in_bom yes) (on_board yes)
+    (property "Reference" "H306" (id 0) (at 261.62 154.94 90)
+      (effects (font (size 1.27 1.27)) (justify left))
+    )
+    (property "Value" "MountingHole" (id 1) (at 264.16 158.75 90)
+      (effects (font (size 1.27 1.27)) (justify left))
+    )
+    (property "Footprint" "MountingHole:MountingHole_2.2mm_M2" (id 2) (at 257.81 153.67 0)
+      (effects (font (size 1.27 1.27)) hide)
+    )
+    (property "Datasheet" "~" (id 3) (at 257.81 153.67 0)
+      (effects (font (size 1.27 1.27)) hide)
+    )
+  )
+  (symbol (lib_id "Mechanical:MountingHole") (at 191.77 153.67 0) (unit 1)
+    (in_bom yes) (on_board yes)
+    (property "Reference" "H301" (id 0) (at 195.58 154.94 90)
+      (effects (font (size 1.27 1.27)) (justify left))
+    )
+    (property "Value" "MountingHole" (id 1) (at 198.12 158.75 90)
+      (effects (font (size 1.27 1.27)) (justify left))
+    )
+    (property "Footprint" "MountingHole:MountingHole_2.2mm_M2" (id 2) (at 191.77 153.67 0)
+      (effects (font (size 1.27 1.27)) hide)
+    )
+    (property "Datasheet" "~" (id 3) (at 191.77 153.67 0)
+      (effects (font (size 1.27 1.27)) hide)
+    )
   )
   (symbol (lib_id "Device:R") (at 222.25 123.19 0) (unit 1)
@@
     (pin "3")
   )
+  (symbol (lib_id "Mechanical:MountingHole") (at 204.47 153.67 0) (unit 1)
+    (in_bom yes) (on_board yes)
+    (property "Reference" "H302" (id 0) (at 208.28 154.94 90)
+      (effects (font (size 1.27 1.27)) (justify left))
+    )
+    (property "Value" "MountingHole" (id 1) (at 210.82 158.75 90)
+      (effects (font (size 1.27 1.27)) (justify left))
+    )
+    (property "Footprint" "MountingHole:MountingHole_2.2mm_M2" (id 2) (at 204.47 153.67 0)
+      (effects (font (size 1.27 1.27)) hide)
+    )
+    (property "Datasheet" "~" (id 3) (at 204.47 153.67 0)
+      (effects (font (size 1.27 1.27)) hide)
+    )
+  )
   (symbol (lib_id "Amplifier_Operational:LM358") (at 172.72 45.72 0) (unit 1)
     (in_bom yes) (on_board yes) (fields_autoplaced)
@@
     (pin "8")
   )
+  (symbol (lib_id "Mechanical:MountingHole") (at 218.44 153.67 0) (unit 1)
+    (in_bom yes) (on_board yes)
+    (property "Reference" "H303" (id 0) (at 222.25 154.94 90)
+      (effects (font (size 1.27 1.27)) (justify left))
+    )
+    (property "Value" "MountingHole" (id 1) (at 224.79 158.75 90)
+      (effects (font (size 1.27 1.27)) (justify left))
+    )
+    (property "Footprint" "MountingHole:MountingHole_2.2mm_M2" (id 2) (at 218.44 153.67 0)
+      (effects (font (size 1.27 1.27)) hide)
+    )
+    (property "Datasheet" "~" (id 3) (at 218.44 153.67 0)
+      (effects (font (size 1.27 1.27)) hide)
+    )
+  )
   (symbol (lib_id "power:GND") (at 265.43 128.27 0) (unit 1)
     (in_bom yes) (on_board yes) (fields_autoplaced)
@@
     (pin "1")
   )
+  (symbol (lib_id "Mechanical:MountingHole") (at 243.84 153.67 0) (unit 1)
+    (in_bom yes) (on_board yes)
+    (property "Reference" "H305" (id 0) (at 247.65 154.94 90)
+      (effects (font (size 1.27 1.27)) (justify left))
+    )
+    (property "Value" "MountingHole" (id 1) (at 250.19 158.75 90)
+      (effects (font (size 1.27 1.27)) (justify left))
+    )
+    (property "Footprint" "MountingHole:MountingHole_2.2mm_M2" (id 2) (at 243.84 153.67 0)
+      (effects (font (size 1.27 1.27)) hide)
+    )
+    (property "Datasheet" "~" (id 3) (at 243.84 153.67 0)
+      (effects (font (size 1.27 1.27)) hide)
+    )
+  )
   (symbol (lib_id "Device:R") (at 252.73 111.76 90) (unit 1)
     (in_bom yes) (on_board yes) (fields_autoplaced)
@@
     (pin "2")
     (pin "3")
+  )
+  (symbol (lib_id "Mechanical:MountingHole") (at 231.14 153.67 0) (unit 1)
+    (in_bom yes) (on_board yes)
+    (property "Reference" "H304" (id 0) (at 234.95 154.94 90)
+      (effects (font (size 1.27 1.27)) (justify left))
+    )
+    (property "Value" "MountingHole" (id 1) (at 237.49 158.75 90)
+      (effects (font (size 1.27 1.27)) (justify left))
+    )
+    (property "Footprint" "MountingHole:MountingHole_2.2mm_M2" (id 2) (at 231.14 153.67 0)
+      (effects (font (size 1.27 1.27)) hide)
+    )
+    (property "Datasheet" "~" (id 3) (at 231.14 153.67 0)
+      (effects (font (size 1.27 1.27)) hide)
+    )
   )
   (symbol (lib_id "Device:Q_NMOS_GDS") (at 195.58 45.72 0) (unit 1)
@@
     (pin "2")
   )
+  (symbol (lib_id "Mechanical:MountingHole") (at 270.51 153.67 0) (unit 1)
+    (in_bom yes) (on_board yes)
+    (property "Reference" "H307" (id 0) (at 274.32 154.94 90)
+      (effects (font (size 1.27 1.27)) (justify left))
+    )
+    (property "Value" "MountingHole" (id 1) (at 276.86 158.75 90)
+      (effects (font (size 1.27 1.27)) (justify left))
+    )
+    (property "Footprint" "MountingHole:MountingHole_2.2mm_M2" (id 2) (at 270.51 153.67 0)
+      (effects (font (size 1.27 1.27)) hide)
+    )
+    (property "Datasheet" "~" (id 3) (at 270.51 153.67 0)
+      (effects (font (size 1.27 1.27)) hide)
+    )
+  )
   (symbol (lib_id "Device:R") (at 90.17 123.19 0) (unit 1)
