File: LedScoreBoard/LedScoreBoard.kicad_sch (KiCad schematic)
At the start: 22 parts

Commit message: 回路図更新
Parts:
- I2C101: renamed from I2C?; footprint (none) -> Connector_PinHeader_2.54mm:PinHeader_1x04_P2.54mm_Vertical
- J101: renamed from J?; footprint (none) -> Connector_PinSocket_2.54mm:PinSocket_1x07_P2.54mm_Vertical
- U102: renamed from U?; footprint RF_Module:MonoWireless_TWE-L-WX -> MonoWireless:MonoWireless_TWELITE-SMD_SMA-Connector
- gave numbers to parts that had none: 19
Connections:
- net MCLR: no longer J101.3 (Pin_3)
- net Vref: now reaches U101.4 (RA2/AN2)
- new net RST: J101.3 (Pin_3)
- no-connect marks 6 -> 21
Other:
- moved on the sheet: J101, SW102, SW103, SW104, SW105, SW106, SW107

Commit message: 配置ブロック決定
Connections:
- net MinusHun: now also U102.2 (DO1/PWM3); no longer U102.7 (DIO5/PWM1)
- net MinusOne: now also U102.7 (DIO5/PWM1); no longer U102.1 (DO0/PWM2)
- net PlusHun: now also U102.1 (DO0/PWM2); no longer U102.6 (DIO4/DO3)
- net PlusOne: now also U102.6 (DIO4/DO3); no longer U102.2 (DO1/PWM3)
Changed lines of the file:
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@@
     (effects (font (size 1.27 1.27)) (justify left bottom))
   )
-  (label "PlusOne" (at 100.33 153.67 0)
+  (label "PlusOne" (at 100.33 143.51 0)
     (effects (font (size 1.27 1.27)) (justify left bottom))
   )
@@
     (effects (font (size 1.27 1.27)) (justify right bottom))
   )
-  (label "PlusHun" (at 100.33 143.51 0)
+  (label "PlusHun" (at 100.33 151.13 0)
     (effects (font (size 1.27 1.27)) (justify left bottom))
   )
@@
     (effects (font (size 1.27 1.27)) (justify right bottom))
   )
-  (label "MinusOne" (at 100.33 151.13 0)
+  (label "MinusOne" (at 100.33 148.59 0)
     (effects (font (size 1.27 1.27)) (justify left bottom))
   )
@@
     (effects (font (size 1.27 1.27)) (justify right bottom))
   )
-  (label "MinusHun" (at 100.33 148.59 0)
+  (label "MinusHun" (at 100.33 153.67 0)
     (effects (font (size 1.27 1.27)) (justify left bottom))
   )
@@
       (reference "U301") (unit 1) (value "LM358") (footprint "Package_SO:TSSOP-8_3x3mm_P0.65mm")
     )
+    (path "/3a5d50f3-7006-4c79-be61-f48c3562ebc1/2dbc7b94-97c3-475d-b979-6be9e5194e4f"
+      (reference "U301") (unit 2) (value "LM358") (footprint "Package_SO:TSSOP-8_3x3mm_P0.65mm")
+    )
+    (path "/3a5d50f3-7006-4c79-be61-f48c3562ebc1/b6b5693a-0427-49e1-a6b6-6fba7bfad11b"
+      (reference "U301") (unit 3) (value "LM358") (footprint "Package_SO:TSSOP-8_3x3mm_P0.65mm")
+    )
     (path "/3a5d50f3-7006-4c79-be61-f48c3562ebc1/49a7e39f-dbf8-48ad-ae14-87294e9b17be"
-      (reference "U301") (unit 2) (value "LM358") (footprint "Package_SO:TSSOP-8_3x3mm_P0.65mm")
-    )
-    (path "/3a5d50f3-7006-4c79-be61-f48c3562ebc1/2dbc7b94-97c3-475d-b979-6be9e5194e4f"
       (reference "U302") (unit 1) (value "LM358") (footprint "Package_SO:TSSOP-8_3x3mm_P0.65mm")
     )
     (path "/3a5d50f3-7006-4c79-be61-f48c3562ebc1/7816d18a-27e2-4b53-9283-eced36a893de"
+      (reference "U302") (unit 2) (value "LM358") (footprint "Package_SO:TSSOP-8_3x3mm_P0.65mm")
+    )
+    (path "/3a5d50f3-7006-4c79-be61-f48c3562ebc1/ab7893e5-bafb-49ed-93d6-a608ebabd528"
+      (reference "U302") (unit 3) (value "LM358") (footprint "Package_SO:TSSOP-8_3x3mm_P0.65mm")
+    )
+    (path "/3a5d50f3-7006-4c79-be61-f48c3562ebc1/6c5994bc-12b4-490c-8a8c-bdca46d1fe70"
       (reference "U303") (unit 1) (value "LM358") (footprint "Package_SO:TSSOP-8_3x3mm_P0.65mm")
     )
     (path "/3a5d50f3-7006-4c79-be61-f48c3562ebc1/6ca03af0-ae49-486a-a25e-abe2ae9a6dc2"
+      (reference "U303") (unit 2) (value "LM358") (footprint "Package_SO:TSSOP-8_3x3mm_P0.65mm")
+    )
+    (path "/3a5d50f3-7006-4c79-be61-f48c3562ebc1/cf418c9d-86e6-4fb6-9327-4965fd456c23"
+      (reference "U303") (unit 3) (value "LM358") (footprint "Package_SO:TSSOP-8_3x3mm_P0.65mm")
+    )
+    (path "/3a5d50f3-7006-4c79-be61-f48c3562ebc1/65a07ce1-182c-4a56-80dd-670515932cc1"
       (reference "U304") (unit 1) (value "LM358") (footprint "Package_SO:TSSOP-8_3x3mm_P0.65mm")
     )
-    (path "/3a5d50f3-7006-4c79-be61-f48c3562ebc1/6c5994bc-12b4-490c-8a8c-bdca46d1fe70"
+    (path "/3a5d50f3-7006-4c79-be61-f48c3562ebc1/b66260a0-15cc-49fa-b1a1-ae2d70ac1cf7"
       (reference "U304") (unit 2) (value "LM358") (footprint "Package_SO:TSSOP-8_3x3mm_P0.65mm")
     )
-    (path "/3a5d50f3-7006-4c79-be61-f48c3562ebc1/b66260a0-15cc-49fa-b1a1-ae2d70ac1cf7"
-      (reference "U305") (unit 1) (value "LM358") (footprint "Package_SO:TSSOP-8_3x3mm_P0.65mm")
-    )
-    (path "/3a5d50f3-7006-4c79-be61-f48c3562ebc1/65a07ce1-182c-4a56-80dd-670515932cc1"
-      (reference "U305") (unit 2) (value "LM358") (footprint "Package_SO:TSSOP-8_3x3mm_P0.65mm")
-    )
-    (path "/3a5d50f3-7006-4c79-be61-f48c3562ebc1/b6b5693a-0427-49e1-a6b6-6fba7bfad11b"
-      (reference "U306") (unit 3) (value "LM358") (footprint "Package_SO:TSSOP-8_3x3mm_P0.65mm")
-    )
-    (path "/3a5d50f3-7006-4c79-be61-f48c3562ebc1/ab7893e5-bafb-49ed-93d6-a608ebabd528"
-      (reference "U307") (unit 3) (value "LM358") (footprint "Package_SO:TSSOP-8_3x3mm_P0.65mm")
-    )
-    (path "/3a5d50f3-7006-4c79-be61-f48c3562ebc1/cf418c9d-86e6-4fb6-9327-4965fd456c23"
-      (reference "U308") (unit 3) (value "LM358") (footprint "Package_SO:TSSOP-8_3x3mm_P0.65mm")
-    )
     (path "/3a5d50f3-7006-4c79-be61-f48c3562ebc1/1bff8d84-01e6-4a04-ba5e-e7976e1c2ef2"
-      (reference "U309") (unit 3) (value "LM358") (footprint "Package_SO:TSSOP-8_3x3mm_P0.65mm")
-    )
-  )
+      (reference "U304") (unit 3) (value "LM358") (footprint "Package_SO:TSSOP-8_3x3mm_P0.65mm")
+    )
+  )

Commit message: パターン完成
Parts:
- added J108: TweLite-R, Connector_PinHeader_2.54mm:PinHeader_1x06_P2.54mm_Vertical, symbol Connector:Conn_01x06_Male
- U102: footprint MonoWireless:MonoWireless_TWELITE-SMD_SMA-Connector -> RF_Module:MonoWireless_TWE-L-WX
Connections:
- net +3.3V: now also J108.6 (Pin_6)
- net GND: now also J108.5 (Pin_5)
- net MCLR: now also J108.1 (Pin_1)
- net MinusHun: now also U102.15 (DIO13/DI2); no longer U102.2 (DO1/PWM3)
- net MinusOne: now also U102.11 (DIO9/DO4); no longer U102.7 (DIO5/PWM1)
- net MinusTen: now also U102.16 (DIO11/DI3); no longer U102.4 (DIO19/DO2)
- net PlusHun: now also U102.13 (DIO12/DI1); no longer U102.1 (DO0/PWM2)
- net PlusOne: now also U102.10 (DIO8/PWM4); no longer U102.6 (DIO4/DO3)
- net PlusTen: now also U102.12 (DIO10/M1); no longer U102.3 (DIO18/DO1)
- net TX: now reaches U102.8 (DIO6/TX)
- net TX: now also J108.4 (Pin_4)
- net RX: now reaches U102.9 (DIO7/RX)
- net RX: now also J108.2 (Pin_2)
- new net PRG: J108.3 (Pin_3), U102.2 (DO1/PWM3)
- no-connect marks 21 -> 18
Other:
- moved on the sheet: I2C101, J107

Commit message: PIC/Twelite書き込み端子ネットリスト修正
Parts:
- U101: value PIC16F1516-ISP -> PIC16F1783
Connections:
- net GND: now also J108.1 (Pin_1); no longer J108.5 (Pin_5)
- net MCLR: now also J108.5 (Pin_5); no longer J108.1 (Pin_1)
- net PGC: now also U101.27 (RB6/ADGRDA/IOC/ICSPCLK/ICDCLK); no longer U101.28 (RB7/ADGRDB/IOC/ICSPDAT/ICDDAT)
- net PGD: now also U101.28 (RB7/ADGRDB/IOC/ICSPDAT/ICDDAT); no longer U101.27 (RB6/ADGRDA/IOC/ICSPCLK/ICDCLK)
- net RX: now also J108.4 (Pin_4); no longer J108.2 (Pin_2)
- net TX: now also J108.2 (Pin_2); no longer J108.4 (Pin_4)

Commit message: Vref修正
Other:
- sheet LedCathodeDrivers ports: added VrefIn; removed Vref
Changed lines of the file:
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@@
       (effects (font (size 1.27 1.27)) (justify right))
-    )
-    (pin "Vref" input (at 191.77 83.82 180)
-      (effects (font (size 1.27 1.27)) (justify left))
     )
     (pin "CsensG" input (at 232.41 111.76 270)
@@
       (effects (font (size 1.27 1.27)) (justify left))
     )
+    (pin "VrefIn" input (at 191.77 83.82 180)
+      (effects (font (size 1.27 1.27)) (justify left))
+    )

Commit message: 回路修正
Parts:
- added R101: 10k, Resistor_SMD:R_0603_1608Metric, symbol Device:R
- added SW102: SW_Push, Button_Switch_THT:SW_PUSH_6mm, symbol Switch:SW_Push
- renumbered J108 to J101, J101 to J102, J107 to J103, J102 to J104, J103 to J105, J104 to J106, J105 to J107, J106 to J108, SW102 to SW103, SW103 to SW104, SW104 to SW105, SW105 to SW106, SW106 to SW107, SW107 to SW108
Connections:
- net +3.3V: now also R101.1
- net GND: now also SW102.2
- net MCLR: no longer J101.5 (Pin_5), U102.21 (~{RESET})
- net RST: no longer names the net of J102.3 (Pin_3)
- net RST: now also R101.2
- new net RESET: J101.5 (Pin_5), SW102.1, U102.21 (~{RESET})

Commit message: ver2完成
Parts:
- removed J107: DC12_IN, TerminalBlock:TerminalBlock_bornier-2_P5.08mm, symbol Connector:Conn_01x02_Male
- added H101, H102, H103, H104: MountingHole, MountingHole:MountingHole_3.2mm_M3, symbol Mechanical:MountingHole
- added H105: MountingHole, MountingHole:MountingHole_6.4mm_M6, symbol Mechanical:MountingHole
- added J107: Conn_01x03_Male, Connector_JST:JST_VH_B3P-VH_1x03_P3.96mm_Vertical, symbol Connector:Conn_01x03_Male
- added R102: 15k, Resistor_SMD:R_0603_1608Metric, symbol Device:R
- added R103: 680, Resistor_SMD:R_0603_1608Metric, symbol Device:R
- added R104, R105: 10k, Resistor_SMD:R_0603_1608Metric, symbol Device:R
- J101: footprint Connector_PinHeader_2.54mm:PinHeader_1x06_P2.54mm_Vertical -> Connector_PinSocket_2.54mm:PinSocket_1x06_P2.54mm_Horizontal
- J103: footprint Connector_PinHeader_2.54mm:PinHeader_1x06_P2.54mm_Vertical -> Connector_PinHeader_2.54mm:PinHeader_1x06_P2.54mm_Horizontal
- J108: value VDD_IN -> Conn_01x02_Male; footprint TerminalBlock:TerminalBlock_bornier-2_P5.08mm -> Connector_PinHeader_2.54mm:PinHeader_1x02_P2.54mm_Vertical
Connections:
- net +12V: now also J107.1 (Pin_1)
- net +3.3V: now also J103.5 (Pin_5), J108.2 (Pin_2), R104.1, R105.1; no longer J101.6 (Pin_6), J103.2 (Pin_2)
- net GND: now also J103.4 (Pin_4), J107.3 (Pin_3), R103.2; no longer J103.3 (Pin_3), J108.2 (Pin_2)
- net MCLR: now also J103.6 (Pin_6); no longer J103.1 (Pin_1)
- net PGC: now also J103.2 (Pin_2); no longer J103.5 (Pin_5)
- net PGD: now also J103.3 (Pin_3); no longer J103.4 (Pin_4)
- net SCL: now also R105.2
- net SDA: now also R104.2
- net VDD: now also J107.2 (Pin_2), R102.1; no longer J108.1 (Pin_1)
- net at U101.25 (RB4/AN11/ADOUT/IOC): now also R102.2, R103.1
- net Vref renamed PicVref
- new net: J101.6 (Pin_6), J108.1 (Pin_1)
- no-connect marks 18 -> 17
Other:
- sheet LedCathodeDrivers ports: added PicVref; removed VrefIn
- moved on the sheet: C102, SW102, U102
